Commit message: Add files via upload

File: ateks_description/urdf/ateks_noetic.urdf (robot description, URDF)
Before this commit: robot ateks, 20 links, 19 joints
Links:
- added link scan_link; collision box size=0.001 0.001 0.001
Joints:
- added joint scan_joint: type fixed, parent base_link, child scan_link, origin xyz=-0.47 -0.2 1.8 rpy=0 0 0, axis 0 0 1
- joint left_wheel_joint: origin xyz=-0.31 -0.325 0.1925 rpy=0 0 0 -> xyz=-0.31 -0.355 0.1925 rpy=0 0 0
- joint right_wheel_joint: origin xyz=-0.31 0.325 0.1925 rpy=0 0 0 -> xyz=-0.31 0.355 0.1925 rpy=0 0 0

Commit message: Some fixes

File: ateks_description/urdf/ateks_noetic.urdf (robot description, URDF)
Before this commit: robot ateks, 21 links, 20 joints
Links:
- link left_wheel: geometry collision cylinder length=0.05 radius=0.17
- link right_wheel: geometry collision cylinder length=0.05 radius=0.17
Joints:
- joint left_wheel_joint: origin xyz=-0.31 -0.355 0.1925 rpy=0 0 0 -> xyz=-0.31 0.335 0.17 rpy=0 0 0
- joint right_wheel_joint: origin xyz=-0.31 0.355 0.1925 rpy=0 0 0 -> xyz=-0.31 -0.335 0.17 rpy=0 0 0
